Commit message: fixed gripper angle publishing

File: katana_description/urdf/katana.urdf.xacro (robot description, xacro)
@@ -168,11 +168,9 @@
       <origin rpy="${rotate} 0 0" xyz="0.034 0 0"/>
       <axis xyz="0 0 1"/>
-      <limit effort="1000.0" lower="-0.44" upper="0.51"  velocity="0.5"/>  <!-- TODO: give correct limits (even lower and upper are not yet correct)  -->
-      <!-- motor 6 limits: lower="-2.085" upper="3.656" (0 is almost closed, fingertips parallel) -->
-      <!-- gemessen: -1.6422866492027579: fully open, 0.17664640984051988: almost closed, fingertips parallel; TODO -->
-    </joint>
+      <limit effort="1000.0" lower="-0.40" upper="0.40"  velocity="0.5"/>  <!-- TODO: give correct limits -->
+   </joint>
     <link name="katana_${prefix}_finger_link">
         <visual>
-          <origin rpy="0 ${M_PI} 0" xyz="-0.034 0 0"/>
+          <origin rpy="0 ${M_PI} 0" xyz="0 0 0"/>
           <geometry>
             <mesh filename="package://katana_description/meshes/katana/katana_gripper_${prefix}_finger.stl"

Commit message: added collision tags

File: katana_description/urdf/katana.urdf.xacro (robot description, xacro)
@@ -6,5 +6,5 @@
        name="katana">
   <property name="scale" value=".001" />               <!-- all katana meshes are scaled in millimeters, but ros uses meters -->
-  <property name="M_PI" value="3.1415926535897931" />  <!-- only approximately correct -->
+  <property name="M_PI" value="3.1415926535897931" />  <!-- only approximately correct ;-) -->
   <!-- all values from the katana manual -->
   <property name="controlbox_height" value="0.08" />
@@ -25,4 +25,11 @@
         </material>
       </visual>
+      <collision>
+        <origin xyz="0 0 0" rpy="0 0 0" />
+        <geometry>
+          <mesh filename="package://katana_description/meshes/katana/katana_internal_controlbox.stl"
+            scale="${scale} ${scale} ${scale}"/>
+        </geometry>
+      </collision>
   </link>
   <joint name="katana_base_joint" type="fixed">
@@ -40,4 +47,11 @@
         <material name="grey" />
       </visual>
+      <collision>
+        <origin xyz="0 0 0" rpy="0 0 ${M_PI}" />
+        <geometry>
+          <mesh filename="package://katana_description/meshes/katana/katana_base_link.stl"
+            scale="${scale} ${scale} ${scale}"/>
+        </geometry>
+      </collision>
   </link>
   <joint name="katana_motor1_pan_joint" type="revolute">
@@ -58,4 +72,11 @@
         <material name="grey" />
       </visual>
+      <collision>
+        <origin xyz="0 0 ${-base_height}" rpy="0 0 0" />
+        <geometry>
+          <mesh filename="package://katana_description/meshes/katana/katana_motor1_pan_link.stl"
+            scale="${scale} ${scale} ${scale}"/>
+        </geometry>
+      </collision>
   </link>
   <joint name="katana_motor2_lift_joint" type="revolute">
@@ -80,4 +101,11 @@
         <material name="grey" />
       </visual>
+      <collision>
+        <origin rpy="${-M_PI/2} 0 0" xyz="0 0 0"/>
+        <geometry>
+          <mesh filename="package://katana_description/meshes/katana/katana_motor2_lift_link.stl"
+            scale="${scale} ${scale} ${scale}"/>
+        </geometry>
+      </collision>
   </link>
   <joint name="katana_motor3_lift_joint" type="revolute">
@@ -102,4 +130,11 @@
         <material name="grey" />
       </visual>
+      <collision>
+        <origin rpy="${-M_PI/2} 0 0" xyz="0 0 0"/>
+        <geometry>
+          <mesh filename="package://katana_description/meshes/katana/katana_motor3_lift_link.stl"
+            scale="${scale} ${scale} ${scale}"/>
+        </geometry>
+      </collision>
   </link>
   <joint name="katana_motor4_lift_joint" type="revolute">
@@ -124,4 +159,11 @@
         <material name="grey" />
       </visual>
+      <collision>
+        <origin rpy="${M_PI/2} 0 0" xyz="0 0 0"/>
+        <geometry>
+          <mesh filename="package://katana_description/meshes/katana/katana_motor4_lift_link.stl"
+            scale="${scale} ${scale} ${scale}"/>
+        </geometry>
+      </collision>
   </link>
   <joint name="katana_motor5_wrist_roll_joint" type="revolute">
@@ -146,4 +188,11 @@
         <material name="grey" />
       </visual>
+      <collision>
+        <origin rpy="0 ${M_PI/2} 0" xyz="0 0 0"/>
+        <geometry>
+          <mesh filename="package://katana_description/meshes/katana/katana_motor5_wrist_roll_link.stl"
+            scale="${scale} ${scale} ${scale}"/>
+        </geometry>
+      </collision>
   </link>
   <joint name="katana_gripper_joint" type="fixed">
@@ -161,4 +210,11 @@
         <material name="grey" />
       </visual>
+      <collision>
+        <origin rpy="0 ${M_PI} 0" xyz="0 0 0"/>
+        <geometry>
+          <mesh filename="package://katana_description/meshes/katana/katana_gripper_link.stl"
+            scale="${scale} ${scale} ${scale}"/>
+        </geometry>
+      </collision>
     </link>
   <xacro:macro name="finger" params="prefix rotate">
@@ -179,4 +235,11 @@
           <material name="grey" />
         </visual>
+        <collision>
+          <origin rpy="0 ${M_PI} 0" xyz="0 0 0"/>
+          <geometry>
+            <mesh filename="package://katana_description/meshes/katana/katana_gripper_${prefix}_finger.stl"
+              scale="${scale} ${scale} ${scale}"/>
+          </geometry>
+        </collision>
     </link>
   </xacro:macro>

Commit message: rescaled all meshes to work around self_filter bug

File: katana_description/urdf/katana.urdf.xacro (robot description, xacro)
@@ -5,5 +5,4 @@
        xmlns:xacro="http://ros.org/wiki/xacro"
        name="katana">
-  <property name="scale" value=".001" />               <!-- all katana meshes are scaled in millimeters, but ros uses meters -->
   <property name="M_PI" value="3.1415926535897931" />  <!-- only approximately correct ;-) -->
   <!-- all values from the katana manual -->
@@ -18,6 +17,5 @@
         <origin xyz="0 0 0" rpy="0 0 0" />
         <geometry>
-          <mesh filename="package://katana_description/meshes/katana/katana_internal_controlbox.stl"
-            scale="${scale} ${scale} ${scale}"/>
+          <mesh filename="package://katana_description/meshes/katana/katana_internal_controlbox.stl" />
         </geometry>
         <material name="grey">
@@ -28,6 +26,5 @@
         <origin xyz="0 0 0" rpy="0 0 0" />
         <geometry>
-          <mesh filename="package://katana_description/meshes/katana/katana_internal_controlbox.stl"
-            scale="${scale} ${scale} ${scale}"/>
+          <mesh filename="package://katana_description/meshes/katana/katana_internal_controlbox.stl" />
         </geometry>
       </collision>
@@ -42,6 +39,5 @@
         <origin xyz="0 0 0" rpy="0 0 ${M_PI}" />
         <geometry>
-          <mesh filename="package://katana_description/meshes/katana/katana_base_link.stl"
-            scale="${scale} ${scale} ${scale}"/>
+          <mesh filename="package://katana_description/meshes/katana/katana_base_link.stl"/>
         </geometry>
         <material name="grey" />
@@ -50,6 +46,5 @@
         <origin xyz="0 0 0" rpy="0 0 ${M_PI}" />
         <geometry>
-          <mesh filename="package://katana_description/meshes/katana/katana_base_link.stl"
-            scale="${scale} ${scale} ${scale}"/>
+          <mesh filename="package://katana_description/meshes/katana/katana_base_link.stl"/>
         </geometry>
       </collision>
@@ -67,6 +62,5 @@
         <origin xyz="0 0 ${-base_height}" rpy="0 0 0" />
         <geometry>
-          <mesh filename="package://katana_description/meshes/katana/katana_motor1_pan_link.stl"
-            scale="${scale} ${scale} ${scale}"/>
+          <mesh filename="package://katana_description/meshes/katana/katana_motor1_pan_link.stl"/>
         </geometry>
         <material name="grey" />
@@ -75,6 +69,5 @@
         <origin xyz="0 0 ${-base_height}" rpy="0 0 0" />
         <geometry>
-          <mesh filename="package://katana_description/meshes/katana/katana_motor1_pan_link.stl"
-            scale="${scale} ${scale} ${scale}"/>
+          <mesh filename="package://katana_description/meshes/katana/katana_motor1_pan_link.stl"/>
         </geometry>
       </collision>
@@ -92,6 +85,5 @@
         <origin rpy="${-M_PI/2} 0 0" xyz="0 0 0"/>
         <geometry>
-          <mesh filename="package://katana_description/meshes/katana/katana_motor2_lift_link.stl"
-            scale="${scale} ${scale} ${scale}"/>
+          <mesh filename="package://katana_description/meshes/katana/katana_motor2_lift_link.stl"/>
         </geometry>
         <!-- <geometry>
@@ -104,6 +96,5 @@
         <origin rpy="${-M_PI/2} 0 0" xyz="0 0 0"/>
         <geometry>
-          <mesh filename="package://katana_description/meshes/katana/katana_motor2_lift_link.stl"
-            scale="${scale} ${scale} ${scale}"/>
+          <mesh filename="package://katana_description/meshes/katana/katana_motor2_lift_link.stl"/>
         </geometry>
       </collision>
@@ -121,6 +112,5 @@
         <origin rpy="${-M_PI/2} 0 0" xyz="0 0 0"/>
         <geometry>
-          <mesh filename="package://katana_description/meshes/katana/katana_motor3_lift_link.stl"
-            scale="${scale} ${scale} ${scale}"/>
+          <mesh filename="package://katana_description/meshes/katana/katana_motor3_lift_link.stl"/>
         </geometry>
          <!--<geometry>
@@ -133,6 +123,5 @@
         <origin rpy="${-M_PI/2} 0 0" xyz="0 0 0"/>
         <geometry>
-          <mesh filename="package://katana_description/meshes/katana/katana_motor3_lift_link.stl"
-            scale="${scale} ${scale} ${scale}"/>
+          <mesh filename="package://katana_description/meshes/katana/katana_motor3_lift_link.stl"/>
         </geometry>
       </collision>
@@ -150,6 +139,5 @@
         <origin rpy="${M_PI/2} 0 0" xyz="0 0 0"/>
         <geometry>
-          <mesh filename="package://katana_description/meshes/katana/katana_motor4_lift_link.stl"
-            scale="${scale} ${scale} ${scale}"/>
+          <mesh filename="package://katana_description/meshes/katana/katana_motor4_lift_link.stl"/>
         </geometry>
          <!-- <geometry>
@@ -162,6 +150,5 @@
         <origin rpy="${M_PI/2} 0 0" xyz="0 0 0"/>
         <geometry>
-          <mesh filename="package://katana_description/meshes/katana/katana_motor4_lift_link.stl"
-            scale="${scale} ${scale} ${scale}"/>
+          <mesh filename="package://katana_description/meshes/katana/katana_motor4_lift_link.stl"/>
         </geometry>
       </collision>
@@ -179,6 +166,5 @@
         <origin rpy="0 ${M_PI/2} 0" xyz="0 0 0"/>
         <geometry>
-          <mesh filename="package://katana_description/meshes/katana/katana_motor5_wrist_roll_link.stl"
-            scale="${scale} ${scale} ${scale}"/>
+          <mesh filename="package://katana_description/meshes/katana/katana_motor5_wrist_roll_link.stl"/>
         </geometry>
          <!--<geometry>
@@ -191,6 +177,5 @@
         <origin rpy="0 ${M_PI/2} 0" xyz="0 0 0"/>
         <geometry>
-          <mesh filename="package://katana_description/meshes/katana/katana_motor5_wrist_roll_link.stl"
-            scale="${scale} ${scale} ${scale}"/>
+          <mesh filename="package://katana_description/meshes/katana/katana_motor5_wrist_roll_link.stl"/>
         </geometry>
       </collision>
@@ -205,6 +190,5 @@
         <origin rpy="0 ${M_PI} 0" xyz="0 0 0"/>
         <geometry>
-          <mesh filename="package://katana_description/meshes/katana/katana_gripper_link.stl"
-            scale="${scale} ${scale} ${scale}"/>
+          <mesh filename="package://katana_description/meshes/katana/katana_gripper_link.stl"/>
         </geometry>
         <material name="grey" />
@@ -213,6 +197,5 @@
         <origin rpy="0 ${M_PI} 0" xyz="0 0 0"/>
         <geometry>
-          <mesh filename="package://katana_description/meshes/katana/katana_gripper_link.stl"
-            scale="${scale} ${scale} ${scale}"/>
+          <mesh filename="package://katana_description/meshes/katana/katana_gripper_link.stl"/>
         </geometry>
       </collision>
@@ -230,6 +213,5 @@
           <origin rpy="0 ${M_PI} 0" xyz="0 0 0"/>
           <geometry>
-            <mesh filename="package://katana_description/meshes/katana/katana_gripper_${prefix}_finger.stl"
-              scale="${scale} ${scale} ${scale}"/>
+            <mesh filename="package://katana_description/meshes/katana/katana_gripper_${prefix}_finger.stl"/>
           </geometry>
           <material name="grey" />
@@ -238,6 +220,5 @@
           <origin rpy="0 ${M_PI} 0" xyz="0 0 0"/>
           <geometry>
-            <mesh filename="package://katana_description/meshes/katana/katana_gripper_${prefix}_finger.stl"
-              scale="${scale} ${scale} ${scale}"/>
+            <mesh filename="package://katana_description/meshes/katana/katana_gripper_${prefix}_finger.stl"/>
           </geometry>
         </collision>

Commit message: added one intertial tag

File: katana_description/urdf/katana.urdf.xacro (robot description, xacro)
@@ -29,4 +29,11 @@
         </geometry>
       </collision>
+      <inertial>
+        <mass value="0.05" />
+        <origin xyz="0.0 0.0 10.0" />
+        <inertia ixx="1.0" ixy="0.0" ixz="0.0"
+                 iyy="1.0" iyz="0.0"
+                 izz="1.0" />
+      </inertial>
   </link>
   <joint name="katana_base_joint" type="fixed">

Commit message: normalized joint angles in description

File: katana_description/urdf/katana.urdf.xacro (robot description, xacro)
@@ -61,7 +61,7 @@
     <parent link="katana_base_link"/>
     <child link="katana_motor1_pan_link" />
-    <origin xyz="0 0 ${base_height}"/>
-    <axis xyz="0 0 1"/>
-    <limit effort="1000.0" lower="0.120" upper="6.159"  velocity="0.5"/>  <!-- TODO:  give correct effort + velocity limits (lower + upper come from angleOffset, angleRange in config file) -->
+    <origin xyz="0 0 ${base_height}" rpy="0 0 ${M_PI}"/>
+    <axis xyz="0 0 1"/>
+    <limit effort="1000.0" lower="${0.120 - M_PI}" upper="${6.159 - M_PI}"  velocity="0.5"/>  <!-- TODO:  give correct effort + velocity limits (lower + upper come from angleOffset, angleRange in config file) -->
   </joint>
   <link name="katana_motor1_pan_link">
@@ -111,7 +111,7 @@
     <parent link="katana_motor2_lift_link" />
     <child  link="katana_motor3_lift_link" />
-    <origin xyz="${link2_length} 0 0" rpy="0 0 ${M_PI}"/>
-    <axis xyz="0 0 1"/>
-    <limit effort="1000.0" lower="0.935" upper="5.195"  velocity="0.5"/>  <!-- TODO: give correct limits -->
+    <origin xyz="${link2_length} 0 0" rpy="0 0 0"/>
+    <axis xyz="0 0 1"/>
+    <limit effort="1000.0" lower="${0.935 - M_PI}" upper="${5.195 - M_PI}"  velocity="0.5"/>  <!-- TODO: give correct limits -->
   </joint>
   <link name="katana_motor3_lift_link">
@@ -138,7 +138,7 @@
     <parent link="katana_motor3_lift_link" />
     <child  link="katana_motor4_lift_link" />
-    <origin rpy="${M_PI} 0 ${M_PI}" xyz="${link3_length} 0 0"/>
-    <axis xyz="0 0 1"/>
-    <limit effort="1000.0" lower="1.116" upper="5.017"  velocity="0.5"/>  <!-- TODO: give correct limits -->
+    <origin rpy="${M_PI} 0 0" xyz="${link3_length} 0 0"/>
+    <axis xyz="0 0 1"/>
+    <limit effort="1000.0" lower="${1.116 - M_PI}" upper="${5.017 - M_PI}"  velocity="0.5"/>  <!-- TODO: give correct limits -->
   </joint>
   <link name="katana_motor4_lift_link">
@@ -165,7 +165,7 @@
     <parent link="katana_motor4_lift_link" />
     <child  link="katana_motor5_wrist_roll_link" />
-    <origin rpy="${-M_PI/2} 0 ${M_PI/2}" xyz="${link4_length} 0 0"/>
-    <axis xyz="0 0 1"/>
-    <limit effort="1000.0" lower="0.152" upper="6.159"  velocity="0.5"/>  <!-- TODO: give correct limits -->
+    <origin rpy="${M_PI/2} 0 ${-M_PI/2}" xyz="${link4_length} 0 0"/>
+    <axis xyz="0 0 1"/>
+    <limit effort="1000.0" lower="${0.152 - M_PI}" upper="${6.159 - M_PI}"  velocity="0.5"/>  <!-- TODO: give correct limits -->
   </joint>
   <link name="katana_motor5_wrist_roll_link">

Commit message: tuned gripper parameters

File: katana_description/urdf/katana.urdf.xacro (robot description, xacro)
@@ -214,5 +214,5 @@
       <origin rpy="${rotate} 0 0" xyz="0.034 0 0"/>
       <axis xyz="0 0 1"/>
-      <limit effort="1000.0" lower="-0.40" upper="0.40"  velocity="0.5"/>  <!-- TODO: give correct limits -->
+      <limit effort="1000.0" lower="-0.44" upper="0.30"  velocity="0.5"/>  <!-- TODO: give correct limits -->
    </joint>
     <link name="katana_${prefix}_finger_link">

Commit message: fixed joint limits in urdf

File: katana_description/urdf/katana.urdf.xacro (robot description, xacro)
@@ -63,5 +63,5 @@
     <origin xyz="0 0 ${base_height}" rpy="0 0 ${M_PI}"/>
     <axis xyz="0 0 1"/>
-    <limit effort="1000.0" lower="${0.120 - M_PI}" upper="${6.159 - M_PI}"  velocity="0.5"/>  <!-- TODO:  give correct effort + velocity limits (lower + upper come from angleOffset, angleRange in config file) -->
+    <limit effort="1000.0" lower="-3.025528" upper="2.891097"  velocity="0.5"/>  <!-- TODO:  give correct effort + velocity limits (lower + upper come from GetEncoderMinPos(), GetEncoderMaxPos()) -->
   </joint>
   <link name="katana_motor1_pan_link">
@@ -86,5 +86,5 @@
     <origin xyz="0 0 0" rpy="${M_PI/2} 0 0"/>
     <axis xyz="0 0 1"/>
-    <limit effort="1000.0" lower="-0.134" upper="2.163"  velocity="0.5"/>  <!-- TODO: give correct limits -->
+    <limit effort="1000.0" lower="-0.135228" upper="2.168572"  velocity="0.5"/>  <!-- TODO: give correct effort + velocity limits -->
   </joint>
   <link name="katana_motor2_lift_link">
@@ -113,5 +113,5 @@
     <origin xyz="${link2_length} 0 0" rpy="0 0 0"/>
     <axis xyz="0 0 1"/>
-    <limit effort="1000.0" lower="${0.935 - M_PI}" upper="${5.195 - M_PI}"  velocity="0.5"/>  <!-- TODO: give correct limits -->
+    <limit effort="1000.0" lower="-2.221804" upper="2.054223"  velocity="0.5"/>  <!-- TODO: give correct effort + velocity limits -->
   </joint>
   <link name="katana_motor3_lift_link">
@@ -140,5 +140,5 @@
     <origin rpy="${M_PI} 0 0" xyz="${link3_length} 0 0"/>
     <axis xyz="0 0 1"/>
-    <limit effort="1000.0" lower="${1.116 - M_PI}" upper="${5.017 - M_PI}"  velocity="0.5"/>  <!-- TODO: give correct limits -->
+    <limit effort="1000.0" lower="-2.033309" upper="1.876133"  velocity="0.5"/>  <!-- TODO: give correct effort + velocity limits -->
   </joint>
   <link name="katana_motor4_lift_link">
@@ -167,5 +167,5 @@
     <origin rpy="${M_PI/2} 0 ${-M_PI/2}" xyz="${link4_length} 0 0"/>
     <axis xyz="0 0 1"/>
-    <limit effort="1000.0" lower="${0.152 - M_PI}" upper="${6.159 - M_PI}"  velocity="0.5"/>  <!-- TODO: give correct limits -->
+    <limit effort="1000.0" lower="-2.993240" upper="2.870985"  velocity="0.5"/>  <!-- TODO: give correct effort + velocity limits -->
   </joint>
   <link name="katana_motor5_wrist_roll_link">
@@ -214,5 +214,5 @@
       <origin rpy="${rotate} 0 0" xyz="0.034 0 0"/>
       <axis xyz="0 0 1"/>
-      <limit effort="1000.0" lower="-0.44" upper="0.30"  velocity="0.5"/>  <!-- TODO: give correct limits -->
+      <limit effort="1000.0" lower="-0.44" upper="0.30"  velocity="0.5"/>  <!-- TODO: give correct effort + velocity limits -->
    </joint>
     <link name="katana_${prefix}_finger_link">

Commit message: using correct velocity and acceleration limits

File: katana_description/urdf/katana.urdf.xacro (robot description, xacro)
@@ -5,5 +5,5 @@
        xmlns:xacro="http://ros.org/wiki/xacro"
        name="katana">
-  <property name="M_PI" value="3.1415926535897931" />  <!-- only approximately correct ;-) -->
+  <property name="M_PI" value="3.1415926535897931" />
   <!-- all values from the katana manual -->
   <property name="controlbox_height" value="0.08" />
@@ -63,5 +63,8 @@
     <origin xyz="0 0 ${base_height}" rpy="0 0 ${M_PI}"/>
     <axis xyz="0 0 1"/>
-    <limit effort="1000.0" lower="-3.025528" upper="2.891097"  velocity="0.5"/>  <!-- TODO:  give correct effort + velocity limits (lower + upper come from GetEncoderMinPos(), GetEncoderMaxPos()) -->
+    <!-- lower + upper limit have been calculated using the KNI's GetEncoderMinPos(), GetEncoderMaxPos();
+         the velocity limit has been calculated by vel_enc2rad(180); 180 encoders / 10ms is the maximum
+         speed limit for all joints, according to the Katana 4D documentation -->
+    <limit effort="1000.0" lower="-3.025528" upper="2.891097" velocity="2.208932"/>  <!-- TODO:  give correct effort limits -->
   </joint>
   <link name="katana_motor1_pan_link">
@@ -86,5 +89,5 @@
     <origin xyz="0 0 0" rpy="${M_PI/2} 0 0"/>
     <axis xyz="0 0 1"/>
-    <limit effort="1000.0" lower="-0.135228" upper="2.168572"  velocity="0.5"/>  <!-- TODO: give correct effort + velocity limits -->
+    <limit effort="1000.0" lower="-0.135228" upper="2.168572"  velocity="1.190799"/>  <!-- TODO: give correct effort limits -->
   </joint>
   <link name="katana_motor2_lift_link">
@@ -113,5 +116,6 @@
     <origin xyz="${link2_length} 0 0" rpy="0 0 0"/>
     <axis xyz="0 0 1"/>
-    <limit effort="1000.0" lower="-2.221804" upper="2.054223"  velocity="0.5"/>  <!-- TODO: give correct effort + velocity limits -->
+    <!-- unexplicably, the measured velocity limit of this motor is exactly half of what vel_enc2rad(180) says -->
+    <limit effort="1000.0" lower="-2.221804" upper="2.054223"  velocity="1.190799"/>  <!-- TODO: give correct effort limits -->
   </joint>
   <link name="katana_motor3_lift_link">
@@ -140,5 +144,5 @@
     <origin rpy="${M_PI} 0 0" xyz="${link3_length} 0 0"/>
     <axis xyz="0 0 1"/>
-    <limit effort="1000.0" lower="-2.033309" upper="1.876133"  velocity="0.5"/>  <!-- TODO: give correct effort + velocity limits -->
+    <limit effort="1000.0" lower="-2.033309" upper="1.876133"  velocity="2.208932"/>  <!-- TODO: give correct effort limits -->
   </joint>
   <link name="katana_motor4_lift_link">
@@ -167,5 +171,5 @@
     <origin rpy="${M_PI/2} 0 ${-M_PI/2}" xyz="${link4_length} 0 0"/>
     <axis xyz="0 0 1"/>
-    <limit effort="1000.0" lower="-2.993240" upper="2.870985"  velocity="0.5"/>  <!-- TODO: give correct effort + velocity limits -->
+    <limit effort="1000.0" lower="-2.993240" upper="2.870985"  velocity="2.208932"/>  <!-- TODO: give correct effort limits -->
   </joint>
   <link name="katana_motor5_wrist_roll_link">
@@ -214,5 +218,5 @@
       <origin rpy="${rotate} 0 0" xyz="0.034 0 0"/>
       <axis xyz="0 0 1"/>
-      <limit effort="1000.0" lower="-0.44" upper="0.30"  velocity="0.5"/>  <!-- TODO: give correct effort + velocity limits -->
+      <limit effort="1000.0" lower="-0.44" upper="0.30"  velocity="0.718834"/>  <!-- TODO: give correct effort limits -->
    </joint>
     <link name="katana_${prefix}_finger_link">
@@ -251,5 +255,5 @@
   </joint>
   <link name="katana_base_frame">
-    <!-- This is the reference coordinate system of the arm (all IK etc. are specified
+    <!-- This is the reference coordinate system of the arm (the KNI kinematics are specified
          in this frame); there is no actual arm part attached to this link -->
   </link>
