Commit message: added effort limits to URDF

File: katana_description/urdf/gazebo.urdf.xacro (robot description, xacro)
@@ -18,5 +18,5 @@
       <l_finger_joint>katana_l_finger_joint</l_finger_joint>
       <updateRate>1000.0</updateRate>
-      <max_torque>10.0</max_torque>  <!-- TODO: find out sensible default; 0.1? -->
+      <max_torque>0.1</max_torque>
     </controller:gazebo_ros_katana_gripper>
   </gazebo>

File: katana_description/urdf/katana.urdf.xacro (robot description, xacro)
@@ -17,4 +17,9 @@
   <!-- All inertial values (mass, center of mass and inertia tensor) have been
        calculated from the meshes using MeshLab -->
+  <!-- lower + upper joint limits have been calculated using the KNI's GetEncoderMinPos(), GetEncoderMaxPos();
+       the velocity limit has been calculated by vel_enc2rad(180); 180 encoders / 10ms is the maximum
+       speed limit for all joints, according to the Katana 4D documentation -->
+  <!-- the effort limits have been measured experimentally from the maximum effort the Gazebo controller
+       uses in normal conditions -->
   <link name="katana_internal_controlbox_link">
     <visual>
@@ -74,8 +79,5 @@
     <origin xyz="0 0 ${base_height}" rpy="0 0 ${M_PI}"/>
     <axis xyz="0 0 1"/>
-    <!-- lower + upper limit have been calculated using the KNI's GetEncoderMinPos(), GetEncoderMaxPos();
-         the velocity limit has been calculated by vel_enc2rad(180); 180 encoders / 10ms is the maximum
-         speed limit for all joints, according to the Katana 4D documentation -->
-    <limit effort="1000.0" lower="-3.025528" upper="2.891097" velocity="2.208932"/>  <!-- TODO:  give correct effort limits -->
+    <limit effort="1.5" lower="-3.025528" upper="2.891097" velocity="2.208932"/>
   </joint>
   <link name="katana_motor1_pan_link">
@@ -107,5 +109,5 @@
     <origin xyz="0 0 0" rpy="${M_PI/2} 0 0"/>
     <axis xyz="0 0 1"/>
-    <limit effort="1000.0" lower="-0.135228" upper="2.168572"  velocity="1.190799"/>  <!-- TODO: give correct effort limits -->
+    <limit effort="0.6" lower="-0.135228" upper="2.168572"  velocity="1.190799"/>
   </joint>
   <link name="katana_motor2_lift_link">
@@ -142,5 +144,5 @@
     <axis xyz="0 0 1"/>
     <!-- unexplicably, the measured velocity limit of this motor is exactly half of what vel_enc2rad(180) says -->
-    <limit effort="1000.0" lower="-2.221804" upper="2.054223"  velocity="1.190799"/>  <!-- TODO: give correct effort limits -->
+    <limit effort="0.25" lower="-2.221804" upper="2.054223"  velocity="1.190799"/>
   </joint>
   <link name="katana_motor3_lift_link">
@@ -176,5 +178,5 @@
     <origin rpy="${M_PI} 0 0" xyz="${link3_length} 0 0"/>
     <axis xyz="0 0 1"/>
-    <limit effort="1000.0" lower="-2.033309" upper="1.876133"  velocity="2.208932"/>  <!-- TODO: give correct effort limits -->
+    <limit effort="0.1" lower="-2.033309" upper="1.876133"  velocity="2.208932"/>
   </joint>
   <link name="katana_motor4_lift_link">
@@ -210,5 +212,5 @@
     <origin rpy="${M_PI/2} 0 ${-M_PI/2}" xyz="${link4_length} 0 0"/>
     <axis xyz="0 0 1"/>
-    <limit effort="1000.0" lower="-2.993240" upper="2.870985"  velocity="2.208932"/>  <!-- TODO: give correct effort limits -->
+    <limit effort="0.01" lower="-2.993240" upper="2.870985"  velocity="2.208932"/>
   </joint>
   <link name="katana_motor5_wrist_roll_link">
@@ -270,5 +272,5 @@
       <origin rpy="${rotate} 0 0" xyz="0.034 0 0"/>
       <axis xyz="0 0 1"/>
-      <limit effort="1000.0" lower="-0.44" upper="0.30"  velocity="0.718834"/>  <!-- TODO: give correct effort limits -->
+      <limit effort="0.1" lower="-0.44" upper="0.30"  velocity="0.718834"/>
    </joint>
     <link name="katana_${prefix}_finger_link">

Commit message: increased max_torque for gripper again
with the previous values, the controller became unstable, funny Gazebo
hopping again :-)

File: katana_description/urdf/gazebo.urdf.xacro (robot description, xacro)
@@ -18,5 +18,5 @@
       <l_finger_joint>katana_l_finger_joint</l_finger_joint>
       <updateRate>1000.0</updateRate>
-      <max_torque>0.1</max_torque>
+      <max_torque>0.5</max_torque>
     </controller:gazebo_ros_katana_gripper>
   </gazebo>

File: katana_description/urdf/katana.urdf.xacro (robot description, xacro)
@@ -272,5 +272,5 @@
       <origin rpy="${rotate} 0 0" xyz="0.034 0 0"/>
       <axis xyz="0 0 1"/>
-      <limit effort="0.1" lower="-0.44" upper="0.30"  velocity="0.718834"/>
+      <limit effort="0.5" lower="-0.44" upper="0.30"  velocity="0.718834"/>
    </joint>
     <link name="katana_${prefix}_finger_link">

Commit message: split out controlbox from Katana URDF

File: katana_description/urdf/gazebo.urdf.xacro (robot description, xacro)
@@ -24,7 +24,4 @@
   <!-- all materials are listed here: simulator_gazebo/gazebo/gazebo/share/gazebo/Media/materials/ -->
   <!-- *************** links *************** -->
-  <gazebo reference="katana_internal_controlbox_link">
-    <material value="PR2/Grey1" />
-  </gazebo>
   <gazebo reference="katana_base_link">
     <material value="PR2/Grey1" />

File: katana_description/urdf/katana_300_6m180.urdf.xacro (robot description, xacro)
@@ -4,10 +4,9 @@
   xmlns:interface="http://playerstage.sourceforge.net/gazebo/xmlschema/#interface"
   xmlns:xacro="http://ros.org/wiki/xacro"
-  name="katana">
+  name="katana_300_6m180">
   <include filename="$(find katana_description)/urdf/transmissions.urdf.xacro"/>
   <include filename="$(find katana_description)/urdf/gazebo.urdf.xacro"/>
   <property name="M_PI" value="3.1415926535897931" />
   <!-- all values from the katana manual -->
-  <property name="controlbox_height" value="0.08" />
   <property name="base_height" value="0.2015" />
   <property name="link2_length" value="0.19" />
@@ -22,40 +21,13 @@
   <!-- the effort limits have been measured experimentally from the maximum effort the Gazebo controller
        uses in normal conditions -->
-  <link name="katana_internal_controlbox_link">
+  <link name="katana_base_link">
     <visual>
       <origin xyz="0 0 0" rpy="0 0 0" />
       <geometry>
-        <mesh filename="package://katana_description/meshes/katana/katana_internal_controlbox.stl" />
+        <mesh filename="package://katana_description/meshes/katana/katana_base_link.stl"/>
       </geometry>
       <material name="grey">
         <color rgba="0.8 0.8 0.8 1"/>
       </material>
-    </visual>
-    <collision>
-      <origin xyz="0 0 0" rpy="0 0 0" />
-      <geometry>
-        <mesh filename="package://katana_description/meshes/katana/convex/katana_internal_controlbox_convex.stlb" />
-      </geometry>
-    </collision>
-    <inertial>
-      <mass value="4.47057045" />
-      <origin xyz="0.000024 -0.006508 0.030555" />
-      <inertia ixx="0.013760086" ixy="-0.000000539" ixz="-0.000000442"
-        iyy="0.015251808" iyz="0.000361753"
-        izz="0.023409309" />
-    </inertial>
-  </link>
-  <joint name="katana_base_joint" type="fixed">
-    <parent link="katana_internal_controlbox_link"/>
-    <child link="katana_base_link"/>
-    <origin xyz="0 0 ${controlbox_height}"/>
-  </joint>
-  <link name="katana_base_link">
-    <visual>
-      <origin xyz="0 0 0" rpy="0 0 0" />
-      <geometry>
-        <mesh filename="package://katana_description/meshes/katana/katana_base_link.stl"/>
-      </geometry>
-      <material name="grey" />
     </visual>
     <collision>

File: katana_description/urdf/katana_450_6m90a.urdf.xacro (robot description, xacro)
@@ -4,10 +4,9 @@
        xmlns:interface="http://playerstage.sourceforge.net/gazebo/xmlschema/#interface"
        xmlns:xacro="http://ros.org/wiki/xacro"
-       name="katana">
+       name="katana_450_6m90a">
   <include filename="$(find katana_description)/urdf/transmissions.urdf.xacro"/>
   <include filename="$(find katana_description)/urdf/gazebo.urdf.xacro"/>
   <property name="M_PI" value="3.1415926535897931" />
   <!-- all values from the katana manual -->
-  <property name="controlbox_height" value="0.08" />
   <property name="base_height" value="0.2015" />
   <property name="link2_length" value="0.19" />
@@ -22,40 +21,13 @@
   <!-- the effort limits have been measured experimentally from the maximum effort the Gazebo controller
        uses in normal conditions -->
-  <link name="katana_internal_controlbox_link">
+  <link name="katana_base_link">
     <visual>
-      <origin xyz="0 0 0" rpy="0 0 0" />
-      <geometry>
-        <mesh filename="package://katana_description/meshes/katana/katana_internal_controlbox.stl" />
+      <origin xyz="0 0 0" rpy="0 0 ${M_PI}" />
+      <geometry>
+        <mesh filename="package://katana_description/meshes/katana/katana_base_link.stl"/>
       </geometry>
       <material name="grey">
         <color rgba="0.8 0.8 0.8 1"/>
       </material>
-    </visual>
-    <collision>
-      <origin xyz="0 0 0" rpy="0 0 0" />
-      <geometry>
-        <mesh filename="package://katana_description/meshes/katana/convex/katana_internal_controlbox_convex.stlb" />
-      </geometry>
-    </collision>
-    <inertial>
-      <mass value="4.47057045" />
-      <origin xyz="0.000024 -0.006508 0.030555" />
-      <inertia ixx="0.013760086" ixy="-0.000000539" ixz="-0.000000442"
-        iyy="0.015251808" iyz="0.000361753"
-        izz="0.023409309" />
-    </inertial>
-  </link>
-  <joint name="katana_base_joint" type="fixed">
-    <parent link="katana_internal_controlbox_link"/>
-    <child link="katana_base_link"/>
-    <origin xyz="0 0 ${controlbox_height}"/>
-  </joint>
-  <link name="katana_base_link">
-    <visual>
-      <origin xyz="0 0 0" rpy="0 0 ${M_PI}" />
-      <geometry>
-        <mesh filename="package://katana_description/meshes/katana/katana_base_link.stl"/>
-      </geometry>
-      <material name="grey" />
     </visual>
     <collision>
