Commit message: rotated katana_base_link to point forward
- also put coke can on other side
- recreated collada files for changed urdf files

File: katana_description/urdf/controlbox.urdf.xacro (robot description, xacro)
@@ -5,5 +5,5 @@
   <link name="katana_internal_controlbox_link">
     <visual>
-      <origin xyz="0 0 0" rpy="0 0 0" />
+      <origin xyz="0 0 0" rpy="0 0 ${M_PI}" />
       <geometry>
         <mesh filename="package://katana_description/meshes/katana/katana_internal_controlbox.stl" />
@@ -14,5 +14,5 @@
     </visual>
     <collision>
-      <origin xyz="0 0 0" rpy="0 0 0" />
+      <origin xyz="0 0 0" rpy="0 0 ${M_PI}" />
       <geometry>
         <mesh filename="package://katana_description/meshes/katana/convex/katana_internal_controlbox_convex.stlb" />

File: katana_description/urdf/katana_300_6m180.urdf.xacro (robot description, xacro)
@@ -285,5 +285,5 @@
     <parent link="katana_base_link"/>
     <child link="katana_base_frame" />
-    <origin xyz="0 0 ${base_height}" rpy="0 0 ${M_PI}"/>
+    <origin xyz="0 0 ${base_height}" rpy="0 0 0"/>
   </joint>
   <link name="katana_base_frame">

File: katana_description/urdf/katana_450_6m90a.urdf.xacro (robot description, xacro)
@@ -23,5 +23,5 @@
   <link name="katana_base_link">
     <visual>
-      <origin xyz="0 0 0" rpy="0 0 ${M_PI}" />
+      <origin xyz="0 0 0" rpy="0 0 0" />
       <geometry>
         <mesh filename="package://katana_description/meshes/katana/katana_base_link.stl"/>
@@ -32,5 +32,5 @@
     </visual>
     <collision>
-      <origin xyz="0 0 0" rpy="0 0 ${M_PI}" />
+      <origin xyz="0 0 0" rpy="0 0 0" />
       <geometry>
         <mesh filename="package://katana_description/meshes/katana/convex/katana_base_link_convex.stlb"/>
@@ -49,5 +49,5 @@
     <parent link="katana_base_link"/>
     <child link="katana_motor1_pan_link" />
-    <origin xyz="0 0 ${base_height}" rpy="0 0 ${M_PI}"/>
+    <origin xyz="0 0 ${base_height}" rpy="0 0 0"/>
     <axis xyz="0 0 1"/>
     <limit effort="1.5" lower="-3.025528" upper="2.891097" velocity="2.208932"/>
@@ -285,5 +285,5 @@
     <parent link="katana_base_link"/>
     <child link="katana_base_frame" />
-    <origin xyz="0 0 ${base_height}" rpy="0 0 ${M_PI}"/>
+    <origin xyz="0 0 ${base_height}" rpy="0 0 0"/>
   </joint>
   <link name="katana_base_frame">

Commit message: katana_description: make Fuerte compatible
copy *.stlb files to *.stl so that Gazebo 1.0 doesn't complain about
"Invalid mesh filename extension"

File: katana_description/urdf/controlbox.urdf.xacro (robot description, xacro)
@@ -16,5 +16,5 @@
       <origin xyz="0 0 0" rpy="0 0 ${M_PI}" />
       <geometry>
-        <mesh filename="package://katana_description/meshes/katana/convex/katana_internal_controlbox_convex.stlb" />
+        <mesh filename="package://katana_description/meshes/katana/convex/katana_internal_controlbox_convex.stl" />
       </geometry>
     </collision>

File: katana_description/urdf/katana_300_6m180.urdf.xacro (robot description, xacro)
@@ -34,5 +34,5 @@
       <origin xyz="0 0 0" rpy="0 0 0" />
       <geometry>
-        <mesh filename="package://katana_description/meshes/katana/convex/katana_base_link_convex.stlb"/>
+        <mesh filename="package://katana_description/meshes/katana/convex/katana_base_link_convex.stl"/>
       </geometry>
     </collision>
@@ -64,5 +64,5 @@
       <origin xyz="0 0 ${-base_height}" rpy="0 0 0" />
       <geometry>
-        <mesh filename="package://katana_description/meshes/katana/convex/katana_motor1_pan_link_convex.stlb"/>
+        <mesh filename="package://katana_description/meshes/katana/convex/katana_motor1_pan_link_convex.stl"/>
       </geometry>
     </collision>
@@ -98,5 +98,5 @@
         <origin rpy="${-M_PI/2} 0 0" xyz="0 0 0"/>
         <geometry>
-          <mesh filename="package://katana_description/meshes/katana/convex/katana_motor2_lift_link_convex.stlb"/>
+          <mesh filename="package://katana_description/meshes/katana/convex/katana_motor2_lift_link_convex.stl"/>
         </geometry>
       </collision>
@@ -133,5 +133,5 @@
         <origin rpy="${-M_PI/2} 0 0" xyz="0 0 0"/>
         <geometry>
-          <mesh filename="package://katana_description/meshes/katana/convex/katana_motor3_lift_link_convex.stlb"/>
+          <mesh filename="package://katana_description/meshes/katana/convex/katana_motor3_lift_link_convex.stl"/>
         </geometry>
       </collision>
@@ -167,5 +167,5 @@
         <origin rpy="${M_PI/2} 0 0" xyz="0 0 0"/>
         <geometry>
-          <mesh filename="package://katana_description/meshes/katana/convex/katana_motor4_lift_link_convex.stlb"/>
+          <mesh filename="package://katana_description/meshes/katana/convex/katana_motor4_lift_link_convex.stl"/>
         </geometry>
       </collision>
@@ -201,5 +201,5 @@
         <origin rpy="0 ${M_PI} 0" xyz="0 0 0"/>
         <geometry>
-          <mesh filename="package://katana_description/meshes/katana/convex/katana_motor5_wrist_roll_link_convex.stlb"/>
+          <mesh filename="package://katana_description/meshes/katana/convex/katana_motor5_wrist_roll_link_convex.stl"/>
         </geometry>
       </collision>
@@ -228,5 +228,5 @@
         <origin rpy="0 ${M_PI} 0" xyz="0 0 0"/>
         <geometry>
-          <mesh filename="package://katana_description/meshes/katana/convex/katana_gripper_link_convex.stlb"/>
+          <mesh filename="package://katana_description/meshes/katana/convex/katana_gripper_link_convex.stl"/>
         </geometry>
       </collision>
@@ -257,5 +257,5 @@
           <origin rpy="0 ${M_PI} 0" xyz="0 0 0"/>
           <geometry>
-            <mesh filename="package://katana_description/meshes/katana/convex/katana_gripper_${prefix}_finger_convex.stlb"/>
+            <mesh filename="package://katana_description/meshes/katana/convex/katana_gripper_${prefix}_finger_convex.stl"/>
           </geometry>
         </collision>

File: katana_description/urdf/katana_400_6m180.urdf.xacro (robot description, xacro)
@@ -34,5 +34,5 @@
       <origin xyz="0 0 0" rpy="0 0 0" />
       <geometry>
-        <mesh filename="package://katana_description/meshes/katana/convex/katana_base_link_convex.stlb"/>
+        <mesh filename="package://katana_description/meshes/katana/convex/katana_base_link_convex.stl"/>
       </geometry>
     </collision>
@@ -64,5 +64,5 @@
       <origin xyz="0 0 ${-base_height}" rpy="0 0 0" />
       <geometry>
-        <mesh filename="package://katana_description/meshes/katana/convex/katana_motor1_pan_link_convex.stlb"/>
+        <mesh filename="package://katana_description/meshes/katana/convex/katana_motor1_pan_link_convex.stl"/>
       </geometry>
     </collision>
@@ -98,5 +98,5 @@
         <origin rpy="${-M_PI/2} 0 0" xyz="0 0 0"/>
         <geometry>
-          <mesh filename="package://katana_description/meshes/katana/convex/katana_motor2_lift_link_convex.stlb"/>
+          <mesh filename="package://katana_description/meshes/katana/convex/katana_motor2_lift_link_convex.stl"/>
         </geometry>
       </collision>
@@ -133,5 +133,5 @@
         <origin rpy="${-M_PI/2} 0 0" xyz="0 0 0"/>
         <geometry>
-          <mesh filename="package://katana_description/meshes/katana/convex/katana_motor3_lift_link_convex.stlb"/>
+          <mesh filename="package://katana_description/meshes/katana/convex/katana_motor3_lift_link_convex.stl"/>
         </geometry>
       </collision>
@@ -167,5 +167,5 @@
         <origin rpy="${M_PI/2} 0 0" xyz="0 0 0"/>
         <geometry>
-          <mesh filename="package://katana_description/meshes/katana/convex/katana_motor4_lift_link_convex.stlb"/>
+          <mesh filename="package://katana_description/meshes/katana/convex/katana_motor4_lift_link_convex.stl"/>
         </geometry>
       </collision>
@@ -201,5 +201,5 @@
         <origin rpy="0 ${M_PI} 0" xyz="0 0 0"/>
         <geometry>
-          <mesh filename="package://katana_description/meshes/katana/convex/katana_motor5_wrist_roll_link_convex.stlb"/>
+          <mesh filename="package://katana_description/meshes/katana/convex/katana_motor5_wrist_roll_link_convex.stl"/>
         </geometry>
       </collision>
@@ -228,5 +228,5 @@
         <origin rpy="0 ${M_PI} 0" xyz="0 0 0"/>
         <geometry>
-          <mesh filename="package://katana_description/meshes/katana/convex/katana_gripper_link_convex.stlb"/>
+          <mesh filename="package://katana_description/meshes/katana/convex/katana_gripper_link_convex.stl"/>
         </geometry>
       </collision>
@@ -257,5 +257,5 @@
           <origin rpy="0 ${M_PI} 0" xyz="0 0 0"/>
           <geometry>
-            <mesh filename="package://katana_description/meshes/katana/convex/katana_gripper_${prefix}_finger_convex.stlb"/>
+            <mesh filename="package://katana_description/meshes/katana/convex/katana_gripper_${prefix}_finger_convex.stl"/>
           </geometry>
         </collision>

File: katana_description/urdf/katana_450_6m90a.urdf.xacro (robot description, xacro)
@@ -34,5 +34,5 @@
       <origin xyz="0 0 0" rpy="0 0 0" />
       <geometry>
-        <mesh filename="package://katana_description/meshes/katana/convex/katana_base_link_convex.stlb"/>
+        <mesh filename="package://katana_description/meshes/katana/convex/katana_base_link_convex.stl"/>
       </geometry>
     </collision>
@@ -64,5 +64,5 @@
       <origin xyz="0 0 ${-base_height}" rpy="0 0 0" />
       <geometry>
-        <mesh filename="package://katana_description/meshes/katana/convex/katana_motor1_pan_link_convex.stlb"/>
+        <mesh filename="package://katana_description/meshes/katana/convex/katana_motor1_pan_link_convex.stl"/>
       </geometry>
     </collision>
@@ -98,5 +98,5 @@
         <origin rpy="${-M_PI/2} 0 0" xyz="0 0 0"/>
         <geometry>
-          <mesh filename="package://katana_description/meshes/katana/convex/katana_motor2_lift_link_convex.stlb"/>
+          <mesh filename="package://katana_description/meshes/katana/convex/katana_motor2_lift_link_convex.stl"/>
         </geometry>
       </collision>
@@ -133,5 +133,5 @@
         <origin rpy="${-M_PI/2} 0 0" xyz="0 0 0"/>
         <geometry>
-          <mesh filename="package://katana_description/meshes/katana/convex/katana_motor3_lift_link_convex.stlb"/>
+          <mesh filename="package://katana_description/meshes/katana/convex/katana_motor3_lift_link_convex.stl"/>
         </geometry>
       </collision>
@@ -167,5 +167,5 @@
         <origin rpy="${M_PI/2} 0 0" xyz="0 0 0"/>
         <geometry>
-          <mesh filename="package://katana_description/meshes/katana/convex/katana_motor4_lift_link_convex.stlb"/>
+          <mesh filename="package://katana_description/meshes/katana/convex/katana_motor4_lift_link_convex.stl"/>
         </geometry>
       </collision>
@@ -201,5 +201,5 @@
         <origin rpy="0 ${M_PI/2} 0" xyz="0 0 0"/>
         <geometry>
-          <mesh filename="package://katana_description/meshes/katana/convex/katana_motor5_wrist_roll_link_convex.stlb"/>
+          <mesh filename="package://katana_description/meshes/katana/convex/katana_motor5_wrist_roll_link_convex.stl"/>
         </geometry>
       </collision>
@@ -228,5 +228,5 @@
         <origin rpy="0 ${M_PI} 0" xyz="0 0 0"/>
         <geometry>
-          <mesh filename="package://katana_description/meshes/katana/convex/katana_gripper_link_convex.stlb"/>
+          <mesh filename="package://katana_description/meshes/katana/convex/katana_gripper_link_convex.stl"/>
         </geometry>
       </collision>
@@ -257,5 +257,5 @@
           <origin rpy="0 ${M_PI} 0" xyz="0 0 0"/>
           <geometry>
-            <mesh filename="package://katana_description/meshes/katana/convex/katana_gripper_${prefix}_finger_convex.stlb"/>
+            <mesh filename="package://katana_description/meshes/katana/convex/katana_gripper_${prefix}_finger_convex.stl"/>
           </geometry>
         </collision>

File: katana_description/urdf/katana_450_6m90b.urdf.xacro (robot description, xacro)
@@ -34,5 +34,5 @@
       <origin xyz="0 0 0" rpy="0 0 0" />
       <geometry>
-        <mesh filename="package://katana_description/meshes/katana/convex/katana_base_link_convex.stlb"/>
+        <mesh filename="package://katana_description/meshes/katana/convex/katana_base_link_convex.stl"/>
       </geometry>
     </collision>
@@ -64,5 +64,5 @@
       <origin xyz="0 0 ${-base_height}" rpy="0 0 0" />
       <geometry>
-        <mesh filename="package://katana_description/meshes/katana/convex/katana_motor1_pan_link_convex.stlb"/>
+        <mesh filename="package://katana_description/meshes/katana/convex/katana_motor1_pan_link_convex.stl"/>
       </geometry>
     </collision>
@@ -98,5 +98,5 @@
         <origin rpy="${-M_PI/2} 0 0" xyz="0 0 0"/>
         <geometry>
-          <mesh filename="package://katana_description/meshes/katana/convex/katana_motor2_lift_link_convex.stlb"/>
+          <mesh filename="package://katana_description/meshes/katana/convex/katana_motor2_lift_link_convex.stl"/>
         </geometry>
       </collision>
@@ -133,5 +133,5 @@
         <origin rpy="${-M_PI/2} 0 0" xyz="0 0 0"/>
         <geometry>
-          <mesh filename="package://katana_description/meshes/katana/convex/katana_motor3_lift_link_convex.stlb"/>
+          <mesh filename="package://katana_description/meshes/katana/convex/katana_motor3_lift_link_convex.stl"/>
         </geometry>
       </collision>
@@ -167,5 +167,5 @@
         <origin rpy="${M_PI/2} 0 0" xyz="0 0 0"/>
         <geometry>
-          <mesh filename="package://katana_description/meshes/katana/convex/katana_motor4_lift_link_convex.stlb"/>
+          <mesh filename="package://katana_description/meshes/katana/convex/katana_motor4_lift_link_convex.stl"/>
         </geometry>
       </collision>
@@ -201,5 +201,5 @@
         <origin rpy="0 ${M_PI/2} 0" xyz="0 0 0"/>
         <geometry>
-          <mesh filename="package://katana_description/meshes/katana/convex/katana_motor5_wrist_roll_link_convex.stlb"/>
+          <mesh filename="package://katana_description/meshes/katana/convex/katana_motor5_wrist_roll_link_convex.stl"/>
         </geometry>
       </collision>
@@ -228,5 +228,5 @@
         <origin rpy="0 ${M_PI} 0" xyz="0 0 0"/>
         <geometry>
-          <mesh filename="package://katana_description/meshes/katana/convex/katana_gripper_link_convex.stlb"/>
+          <mesh filename="package://katana_description/meshes/katana/convex/katana_gripper_link_convex.stl"/>
         </geometry>
       </collision>
@@ -257,5 +257,5 @@
           <origin rpy="0 ${M_PI} 0" xyz="0 0 0"/>
           <geometry>
-            <mesh filename="package://katana_description/meshes/katana/convex/katana_gripper_${prefix}_finger_convex.stlb"/>
+            <mesh filename="package://katana_description/meshes/katana/convex/katana_gripper_${prefix}_finger_convex.stl"/>
           </geometry>
         </collision>

Commit message: changed Gazebo colors to something Gazebo 1.0 knows

File: katana_description/urdf/controlbox.urdf.xacro (robot description, xacro)
@@ -33,5 +33,5 @@
   </joint>
   <gazebo reference="katana_internal_controlbox_link">
-    <material value="PR2/Grey1" />
+    <material value="Gazebo/Grey" />
   </gazebo>
 </robot>

File: katana_description/urdf/gazebo.urdf.xacro (robot description, xacro)
@@ -25,28 +25,28 @@
   <!-- *************** links *************** -->
   <gazebo reference="katana_base_link">
-    <material value="PR2/Grey1" />
+    <material value="Gazebo/Grey" />
   </gazebo>
   <gazebo reference="katana_motor1_pan_link">
-    <material value="PR2/Grey1" />
+    <material value="Gazebo/Grey" />
     <turnGravityOff>true</turnGravityOff>
   </gazebo>
   <gazebo reference="katana_motor2_lift_link">
-    <material value="PR2/Grey1" />
+    <material value="Gazebo/Grey" />
     <turnGravityOff>true</turnGravityOff>
   </gazebo>
   <gazebo reference="katana_motor3_lift_link">
-    <material value="PR2/Grey1" />
+    <material value="Gazebo/Grey" />
     <turnGravityOff>true</turnGravityOff>
   </gazebo>
   <gazebo reference="katana_motor4_lift_link">
-    <material value="PR2/Grey1" />
+    <material value="Gazebo/Grey" />
     <turnGravityOff>true</turnGravityOff>
   </gazebo>
   <gazebo reference="katana_motor5_wrist_roll_link">
-    <material value="PR2/Grey1" />
+    <material value="Gazebo/Grey" />
     <turnGravityOff>true</turnGravityOff>
   </gazebo>
   <gazebo reference="katana_gripper_link">
-    <material value="PR2/Grey1" />
+    <material value="Gazebo/Grey" />
     <turnGravityOff>true</turnGravityOff>
   </gazebo>
@@ -54,5 +54,5 @@
     <!-- TODO: set friction parameters (mu1, mu2, kp, kd) for fingers (see PR2 gripper.gazebo.xacro) -->
     <gazebo reference="katana_${prefix}_finger_link">
-      <material value="PR2/Grey1" />
+      <material value="Gazebo/Grey" />
       <turnGravityOff>true</turnGravityOff>
     </gazebo>
