Commit message: katana_description: fix transmissions with gazebo 3 / indigo
This is backwards compatible.

hardware interface is now a required option of transmission/joint

File: katana_description/urdf/transmissions.urdf.xacro (robot description, xacro)
@@ -5,5 +5,7 @@
     <transmission name="${name}_trans">
       <type>transmission_interface/SimpleTransmission</type>
-      <joint name="${name}_joint" />
+      <joint name="${name}_joint">
+        <hardwareInterface>EffortJointInterface</hardwareInterface>
+      </joint>
       <actuator name="${name}_motor">
         <hardwareInterface>EffortJointInterface</hardwareInterface>
