Commit message: migration to ROS noetic

File: katana_description/urdf/katana_300_6m180.urdf.xacro (robot description, xacro)
@@ -1,14 +1,13 @@
 <?xml version="1.0"?>
-<robot xmlns:xacro="http://ros.org/wiki/xacro"
-  name="katana_300_6m180">
+<robot xmlns:xacro="http://ros.org/wiki/xacro" name="katana_300_6m180">
   <xacro:include filename="$(find katana_description)/urdf/transmissions.urdf.xacro"/>
   <xacro:include filename="$(find katana_description)/urdf/gazebo.urdf.xacro"/>
-  <property name="M_PI" value="3.1415926535897931" />
+  <xacro:property name="M_PI" value="3.1415926535897931" />
   <!-- all values from the katana manual -->
-  <property name="base_height" value="0.2015" />
-  <property name="link2_length" value="0.19" />
-  <property name="link3_length" value="0.139" />
-  <property name="link4_length" value="0.1523" />
-  <property name="link5_length" value="0.1505" />
+  <xacro:property name="base_height" value="0.2015" />
+  <xacro:property name="link2_length" value="0.19" />
+  <xacro:property name="link3_length" value="0.139" />
+  <xacro:property name="link4_length" value="0.1523" />
+  <xacro:property name="link5_length" value="0.1505" />
   <!-- All inertial values (mass, center of mass and inertia tensor) have been
        calculated from the meshes using MeshLab -->

File: katana_description/urdf/katana_300_6m180_with_controlbox.urdf.xacro (robot description, xacro)
@@ -1,5 +1,4 @@
 <?xml version="1.0"?>
-<robot xmlns:xacro="http://ros.org/wiki/xacro"
-  name="katana_300_6m180_with_controlbox">
+<robot xmlns:xacro="http://ros.org/wiki/xacro" name="katana_300_6m180_with_controlbox">
   <xacro:include filename="$(find katana_description)/urdf/controlbox.urdf.xacro"/>
   <xacro:include filename="$(find katana_description)/urdf/katana_300_6m180.urdf.xacro"/>

File: katana_description/urdf/katana_400_6m180.urdf.xacro (robot description, xacro)
@@ -1,14 +1,13 @@
 <?xml version="1.0"?>
-<robot xmlns:xacro="http://ros.org/wiki/xacro"
-  name="katana_400_6m180">
+<robot xmlns:xacro="http://ros.org/wiki/xacro" name="katana_400_6m180">
   <xacro:include filename="$(find katana_description)/urdf/transmissions.urdf.xacro"/>
   <xacro:include filename="$(find katana_description)/urdf/gazebo.urdf.xacro"/>
-  <property name="M_PI" value="3.1415926535897931" />
+  <xacro:property name="M_PI" value="3.1415926535897931" />
   <!-- all values from the katana manual -->
-  <property name="base_height" value="0.2015" />
-  <property name="link2_length" value="0.19" />
-  <property name="link3_length" value="0.139" />
-  <property name="link4_length" value="0.1523" />
-  <property name="link5_length" value="0.1505" />
+  <xacro:property name="base_height" value="0.2015" />
+  <xacro:property name="link2_length" value="0.19" />
+  <xacro:property name="link3_length" value="0.139" />
+  <xacro:property name="link4_length" value="0.1523" />
+  <xacro:property name="link5_length" value="0.1505" />
   <!-- All inertial values (mass, center of mass and inertia tensor) have been
        calculated from the meshes using MeshLab -->

File: katana_description/urdf/katana_400_6m180_with_controlbox.urdf.xacro (robot description, xacro)
@@ -1,5 +1,4 @@
 <?xml version="1.0"?>
-<robot xmlns:xacro="http://ros.org/wiki/xacro"
-  name="katana_400_6m180_with_controlbox">
+<robot xmlns:xacro="http://ros.org/wiki/xacro" name="katana_400_6m180_with_controlbox">
   <xacro:include filename="$(find katana_description)/urdf/controlbox.urdf.xacro"/>
   <xacro:include filename="$(find katana_description)/urdf/katana_400_6m180.urdf.xacro"/>

File: katana_description/urdf/katana_450_6m90a.urdf.xacro (robot description, xacro)
@@ -1,15 +1,14 @@
 <?xml version="1.0"?>
-<robot xmlns:xacro="http://ros.org/wiki/xacro"
-       name="katana_450_6m90a">
-  <xacro:include filename="$(find katana_description)/urdf/transmissions.urdf.xacro"/>
-  <xacro:include filename="$(find katana_description)/urdf/gazebo.urdf.xacro"/>
-  <property name="M_PI" value="3.1415926535897931" />
+<robot xmlns:xacro="http://ros.org/wiki/xacro" name="katana_450_6m90a">
+  <xacro:include filename='$(find katana_description)/urdf/transmissions.urdf.xacro'/>
+  <xacro:include filename='$(find katana_description)/urdf/gazebo.urdf.xacro'/>
+  <xacro:property name="M_PI" value="3.1415926535897931" />
   <!-- all values from the katana manual -->
-  <property name="base_height" value="0.2015" />
-  <property name="link2_length" value="0.19" />
-  <property name="link3_length" value="0.139" />
-  <property name="link4_length" value="0.1473" />
-  <property name="link5_length" value="0.1505" />
-  <property name="tool_frame_offset" value="0.11" />
+  <xacro:property name="base_height" value="0.2015" />
+  <xacro:property name="link2_length" value="0.19" />
+  <xacro:property name="link3_length" value="0.139" />
+  <xacro:property name="link4_length" value="0.1473" />
+  <xacro:property name="link5_length" value="0.1505" />
+  <xacro:property name="tool_frame_offset" value="0.11" />
   <!-- All inertial values (mass, center of mass and inertia tensor) have been
        calculated from the meshes using MeshLab -->

File: katana_description/urdf/katana_450_6m90a_with_controlbox.urdf.xacro (robot description, xacro)
@@ -1,6 +1,5 @@
 <?xml version="1.0"?>
-<robot xmlns:xacro="http://ros.org/wiki/xacro"
-  name="katana_450_6m90a_with_controlbox">
-  <xacro:include filename="$(find katana_description)/urdf/controlbox.urdf.xacro"/>
-  <xacro:include filename="$(find katana_description)/urdf/katana_450_6m90a.urdf.xacro"/>
+<robot xmlns:xacro="http://ros.org/wiki/xacro" name="katana_450_6m90a_with_controlbox">
+  <xacro:include filename='$(find katana_description)/urdf/controlbox.urdf.xacro'/>
+  <xacro:include filename='$(find katana_description)/urdf/katana_450_6m90a.urdf.xacro'/>
 </robot>

File: katana_description/urdf/katana_450_6m90b.urdf.xacro (robot description, xacro)
@@ -1,14 +1,13 @@
 <?xml version="1.0"?>
-<robot xmlns:xacro="http://ros.org/wiki/xacro"
-       name="katana_450_6m90b">
+<robot xmlns:xacro="http://ros.org/wiki/xacro" name="katana_450_6m90b">
   <xacro:include filename="$(find katana_description)/urdf/transmissions.urdf.xacro"/>
   <xacro:include filename="$(find katana_description)/urdf/gazebo.urdf.xacro"/>
-  <property name="M_PI" value="3.1415926535897931" />
+  <xacro:property name="M_PI" value="3.1415926535897931" />
   <!-- all values from the katana manual -->
-  <property name="base_height" value="0.2015" />
-  <property name="link2_length" value="0.19" />
-  <property name="link3_length" value="0.139" />
-  <property name="link4_length" value="0.1473" />
-  <property name="link5_length" value="0.1505" />
+  <xacro:property name="base_height" value="0.2015" />
+  <xacro:property name="link2_length" value="0.19" />
+  <xacro:property name="link3_length" value="0.139" />
+  <xacro:property name="link4_length" value="0.1473" />
+  <xacro:property name="link5_length" value="0.1505" />
   <!-- All inertial values (mass, center of mass and inertia tensor) have been
        calculated from the meshes using MeshLab -->

File: katana_description/urdf/katana_450_6m90b_with_controlbox.urdf.xacro (robot description, xacro)
@@ -1,5 +1,4 @@
 <?xml version="1.0"?>
-<robot xmlns:xacro="http://ros.org/wiki/xacro"
-  name="katana_450_6m90b_with_controlbox">
+<robot xmlns:xacro="http://ros.org/wiki/xacro" name="katana_450_6m90b_with_controlbox">
   <xacro:include filename="$(find katana_description)/urdf/controlbox.urdf.xacro"/>
   <xacro:include filename="$(find katana_description)/urdf/katana_450_6m90b.urdf.xacro"/>
