Commit message: fix indentation

File: kurtana_description/urdf/kinect.urdf.xacro (robot description, xacro)
@@ -1,70 +1,70 @@
 <?xml version="1.0"?>
 <robot xmlns:sensor="http://playerstage.sourceforge.net/gazebo/xmlschema/#sensor"
-       xmlns:controller="http://playerstage.sourceforge.net/gazebo/xmlschema/#controller"
-       xmlns:interface="http://playerstage.sourceforge.net/gazebo/xmlschema/#interface"
-       xmlns:xacro="http://ros.org/wiki/xacro"
-       name="kinect">
-        <property name="M_PI" value="3.1415926535897931" />
- <link name="kinect_link">
- 	<inertial>
- 		<mass value="0.00001" />
- 		<origin xyz="0 0 0" />
- 	    <inertia ixx="1.0" ixy="0.0" ixz="0.0"
- 			iyy="1.0" iyz="0.0"
- 			izz="1.0" />
+  xmlns:controller="http://playerstage.sourceforge.net/gazebo/xmlschema/#controller"
+  xmlns:interface="http://playerstage.sourceforge.net/gazebo/xmlschema/#interface"
+  xmlns:xacro="http://ros.org/wiki/xacro"
+  name="kinect">
+  <property name="M_PI" value="3.1415926535897931" />
+  <link name="kinect_link">
+    <inertial>
+      <mass value="0.00001" />
+      <origin xyz="0 0 0" />
+      <inertia ixx="1.0" ixy="0.0" ixz="0.0"
+        iyy="1.0" iyz="0.0"
+        izz="1.0" />
     </inertial>
- 	<visual>
- 		<origin xyz=" 0 0 0 " rpy="0 0 0" />
- 		<geometry>
-			 <mesh filename="package://kurtana_description/meshes/kinect/kinect.dae"/>
-		</geometry>
- </visual>
- 	<collision>
- 		<origin xyz="0.0 0.0 0.0" rpy="0 0 0" />
- 		<geometry>
- 			<box size="0.0730 .2760 0.0720"/>
- 		</geometry>
- 	</collision>
- </link>
- <joint name="kinect_depth_joint" type="fixed">
- 	<origin xyz="0 0.018 0" rpy="0 0 0" />
- 	<parent link="kinect_link" />
- 	<child link="kinect_depth_origin" />
- </joint>
- <link name="kinect_depth_origin">
- 	<inertial>
- 	<mass value="0.000001" />
- 	<origin xyz="0 0 0" />
-	 <inertia ixx="0.0001" ixy="0.0" ixz="0.0"
- 			  iyy="0.0001" iyz="0.0"
-              izz="0.0001" />
- 	</inertial>
- </link>
- <joint name="kinect_depth_optical_joint" type="fixed">
- 	<origin xyz="0 0 0" rpy="${-M_PI/2} 0 ${-M_PI/2}" />
- 	<parent link="kinect_depth_origin" />
- 	<child link="kinect_depth" />
- </joint>
- <link name="kinect_depth">
- 	<inertial>
- 	<mass value="0.000001" />
-	 <origin xyz="0 0 0" />
-	 	<inertia ixx="0.0001" ixy="0.0" ixz="0.0"
-		 	 iyy="0.0001" iyz="0.0" izz="0.0001" />
- 		</inertial>
- </link>
- <joint name="kinect_rgb_joint" type="fixed">
- 	<origin xyz="0 -0.005 0" rpy="0 0 0" />
- 	<parent link="kinect_link" />
- 	<child link="kinect_rgb" />
- </joint>
- <link name="kinect_rgb">
- 	<inertial>
- 	<mass value="0.000001" />
- 	<origin xyz="0 0 0" />
- 	<inertia ixx="0.0001" ixy="0.0" ixz="0.0"
- 			iyy="0.0001" iyz="0.0"
- 			izz="0.0001" />
-	</inertial>
- </link>
- </robot>
+    <visual>
+      <origin xyz=" 0 0 0 " rpy="0 0 0" />
+      <geometry>
+        <mesh filename="package://kurtana_description/meshes/kinect/kinect.dae"/>
+      </geometry>
+    </visual>
+    <collision>
+      <origin xyz="0.0 0.0 0.0" rpy="0 0 0" />
+      <geometry>
+        <box size="0.0730 .2760 0.0720"/>
+      </geometry>
+    </collision>
+  </link>
+  <joint name="kinect_depth_joint" type="fixed">
+    <origin xyz="0 0.018 0" rpy="0 0 0" />
+    <parent link="kinect_link" />
+    <child link="kinect_depth_origin" />
+  </joint>
+  <link name="kinect_depth_origin">
+    <inertial>
+      <mass value="0.000001" />
+      <origin xyz="0 0 0" />
+      <inertia ixx="0.0001" ixy="0.0" ixz="0.0"
+        iyy="0.0001" iyz="0.0"
+        izz="0.0001" />
+    </inertial>
+  </link>
+  <joint name="kinect_depth_optical_joint" type="fixed">
+    <origin xyz="0 0 0" rpy="${-M_PI/2} 0 ${-M_PI/2}" />
+    <parent link="kinect_depth_origin" />
+    <child link="kinect_depth" />
+  </joint>
+  <link name="kinect_depth">
+    <inertial>
+      <mass value="0.000001" />
+      <origin xyz="0 0 0" />
+      <inertia ixx="0.0001" ixy="0.0" ixz="0.0"
+        iyy="0.0001" iyz="0.0" izz="0.0001" />
+    </inertial>
+  </link>
+  <joint name="kinect_rgb_joint" type="fixed">
+    <origin xyz="0 -0.005 0" rpy="0 0 0" />
+    <parent link="kinect_link" />
+    <child link="kinect_rgb" />
+  </joint>
+  <link name="kinect_rgb">
+    <inertial>
+      <mass value="0.000001" />
+      <origin xyz="0 0 0" />
+      <inertia ixx="0.0001" ixy="0.0" ixz="0.0"
+        iyy="0.0001" iyz="0.0"
+        izz="0.0001" />
+    </inertial>
+  </link>
+</robot>
