Commit message: fix indentation

File: kurtana_description/urdf/kurtana.urdf.xacro (robot description, xacro)
@@ -1,17 +1,17 @@
 <?xml version="1.0"?>
 <robot xmlns:sensor="http://playerstage.sourceforge.net/gazebo/xmlschema/#sensor"
-       xmlns:controller="http://playerstage.sourceforge.net/gazebo/xmlschema/#controller"
-       xmlns:interface="http://playerstage.sourceforge.net/gazebo/xmlschema/#interface"
-       xmlns:xacro="http://ros.org/wiki/xacro"
-       name="kurtana">
+  xmlns:controller="http://playerstage.sourceforge.net/gazebo/xmlschema/#controller"
+  xmlns:interface="http://playerstage.sourceforge.net/gazebo/xmlschema/#interface"
+  xmlns:xacro="http://ros.org/wiki/xacro"
+  name="kurtana">
   <property name="M_PI" value="3.1415926535897931" />
-<!-- ******************** -->
-<!-- *** KURTana Rack *** -->
-<!-- ******************** -->
-<include filename="$(find kurt_description)/parts/kurtana_rack.urdf.xacro" />
-<!-- ************************ -->
-<!-- *** Microsoft Kinect *** -->
-<!-- ************************ -->
- <include filename="$(find kurt_description)/parts/kinect.urdf.xacro" />
+  <!-- ******************** -->
+  <!-- *** KURTana Rack *** -->
+  <!-- ******************** -->
+  <include filename="$(find kurt_description)/parts/kurtana_rack.urdf.xacro" />
+  <!-- ************************ -->
+  <!-- *** Microsoft Kinect *** -->
+  <!-- ************************ -->
+  <include filename="$(find kurt_description)/parts/kinect.urdf.xacro" />
   <joint name="kurtana_kinect_joint" type="fixed">
     <parent link="kurtana_pitchpole_link" />
@@ -19,15 +19,12 @@
     <origin xyz="${0.0730/2} 0 ${0.0720+kinect_gap}" rpy="0 0 0"/>
   </joint>
-<!-- **************************** -->
-<!-- *** Neuronics Katana Arm *** -->
-<!-- **************************** -->
- <include filename="$(find katana_description)/urdf/katana_450_6m90a_with_controlbox.urdf.xacro" />
- <joint name="kurtana_baseplate_controlbox_joint" type="fixed">
- 	<origin xyz="0.05 0 ${baseplate_height*1.5}" rpy="0 0 0" />
- 	<parent link="kurtana_baseplate_link" />
- 	<child link="katana_internal_controlbox_link" />
- </joint>
-<!-- ***************** -->
-<!-- *** Kurt Base *** -->
-<!-- ***************** -->
+  <!-- **************************** -->
+  <!-- *** Neuronics Katana Arm *** -->
+  <!-- **************************** -->
+  <include filename="$(find katana_description)/urdf/katana_450_6m90a_with_controlbox.urdf.xacro" />
+  <joint name="kurtana_baseplate_controlbox_joint" type="fixed">
+    <origin xyz="0.05 0 ${baseplate_height*1.5}" rpy="0 0 0" />
+    <parent link="kurtana_baseplate_link" />
+    <child link="katana_internal_controlbox_link" />
+  </joint>
 </robot>
