Commit message: reduce coke_can.urdf mass so the arm can lift it
This is an evil hack; later the PID gains of the arm should be tuned so
that it can actually lift the can.

File: katana_arm_gazebo/urdf/coke_can.urdf (robot description, URDF)
Before this commit: robot coke_can_model, 1 links, 0 joints
Links:
- link coke_can: mass 0.1 -> 0.001
